File: Lab1/Lab1/Lab1.sch (KiCad schematic (older format))
At the start: 16 parts, among them J1 Conn_01x05_Male, J2 USB_OTG, U1 CMWX1ZZABZ-078, U2 LM1117ADJ

Commit message: Lab 1 DONE
Parts:
- added C10, C9: 10u, Capacitor_SMD:CP_Elec_6.3x7.7, symbol Device:CP
- U2: footprint (none) -> Package_TO_SOT_SMD:SOT-223
Connections:
- net +3V3: now also C10.1
- net GND: now also C10.2, C9.2
- net at C7.2, J2.1 (VBUS), U2.3 (Vin): now also C9.1
Changed lines of the file:
@@
 $EndComp
 Wire Wire Line
-	7950 1850 8050 1850
+	7950 1850 8000 1850
 Wire Wire Line
 	8500 1850 8700 1850
@@
 F 0 "U2" H 9150 1415 50  0000 C CNN
 F 1 "LM1117ADJ" H 9150 1324 50  0000 C CNN
-F 2 "" H 9150 1300 50  0001 C CNN
+F 2 "Package_TO_SOT_SMD:SOT-223" H 9150 1300 50  0001 C CNN
 F 3 "" H 9150 1300 50  0001 C CNN
 	1    9150 1300
@@
 Wire Wire Line
 	8050 1850 8200 1850
+$Comp
+L Device:CP C10
+U 1 1 5E36A307
+P 10350 1900
+F 0 "C10" H 10468 1946 50  0000 L CNN
+F 1 "10u" H 10468 1855 50  0000 L CNN
+F 2 "Capacitor_SMD:CP_Elec_6.3x7.7" H 10388 1750 50  0001 C CNN
+F 3 "~" H 10350 1900 50  0001 C CNN
+	1    10350 1900
+	1    0    0    -1
+$EndComp
+Wire Wire Line
+	10350 1750 10350 1450
+Wire Wire Line
+	10350 1450 10000 1450
+Connection ~ 10000 1450
+Wire Wire Line
+	10350 2050 10350 2600
+Wire Wire Line
+	10350 2600 10000 2600
+Connection ~ 10000 2600
+$Comp
+L Device:CP C9
+U 1 1 5E36F6C9
+P 8350 2250
+F 0 "C9" V 8095 2250 50  0000 C CNN
+F 1 "10u" V 8186 2250 50  0000 C CNN
+F 2 "Capacitor_SMD:CP_Elec_6.3x7.7" H 8388 2100 50  0001 C CNN
+F 3 "~" H 8350 2250 50  0001 C CNN
+	1    8350 2250
+	0    1    1    0
+$EndComp
+Wire Wire Line
+	8500 2250 8700 2250
+Wire Wire Line
+	8700 2250 8700 1850
+Connection ~ 8700 1850
+Wire Wire Line
+	8200 2250 8000 2250
+Wire Wire Line
+	8000 2250 8000 1850
+Connection ~ 8000 1850
+Wire Wire Line
+	8000 1850 8050 1850
 $EndSCHEMATC

Commit message: Lab 2 DONE
Parts:
- U1: footprint RF_Module:CMWX1ZZABZ -> CMWX1ZZABZ:CMWX1ZZABZ_longer_pads
Connections:
- net GND: no longer R3.2, R4.1, U2.1 (ADJ)
- net +5V: now reaches C7.2, C9.1, J2.1 (VBUS), U2.3 (Vin)
- new net: R3.2, R4.1, U2.1 (ADJ)
Changed lines of the file:
@@
 F 0 "U1" H 5650 1961 50  0000 C CNN
 F 1 "CMWX1ZZABZ-078" H 5650 1870 50  0000 C CNN
-F 2 "RF_Module:CMWX1ZZABZ" H 5650 3550 50  0001 C CNN
+F 2 "CMWX1ZZABZ:CMWX1ZZABZ_longer_pads" H 5650 3550 50  0001 C CNN
 F 3 "https://wireless.murata.com/RFM/data/type_abz.pdf" H 8100 2050 50  0001 C CNN
 	1    5650 3550
@@
 $EndComp
 Wire Wire Line
-	8000 950  8400 950
+	8000 950  8200 950
 Wire Wire Line
 	8400 950  8400 1150
@@
 	10000 2600 10000 2050
 Connection ~ 9650 2600
-Wire Wire Line
-	9650 2600 9050 2600
-Wire Wire Line
-	9050 2600 9050 2050
-Connection ~ 9050 2050
 Wire Wire Line
 	3700 3300 3700 2600
@@
 Wire Wire Line
 	8000 1850 8050 1850
+$Comp
+L power:+5V #PWR0112
+U 1 1 5E3B1A8E
+P 8200 850
+F 0 "#PWR0112" H 8200 700 50  0001 C CNN
+F 1 "+5V" H 8215 1023 50  0000 C CNN
+F 2 "" H 8200 850 50  0001 C CNN
+F 3 "" H 8200 850 50  0001 C CNN
+	1    8200 850
+	1    0    0    -1
+$EndComp
+Wire Wire Line
+	8200 850  8200 950
+Connection ~ 8200 950
+Wire Wire Line
+	8200 950  8400 950
 $EndSCHEMATC
